File: rpi-can-rs485-2/rpi-can-rs485.sch (EAGLE design)
At the start: 35 parts, among them IC1 LM555N, IC2 75176AP, U1 MCP2515SO, U3 MCP2551SN, X1 D-SUB9-H5M09RA

Commit message: misc changes
Other:
- note added: "CAN"
- note added: "RS-485 with Auto TX Enable"
- note removed: "2x CAN"
- note removed: "Optically isolated RS-485"
Changed lines of the file:
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@@
 <?xml version="1.0" encoding="utf-8"?>
 <!DOCTYPE eagle SYSTEM "eagle.dtd">
-<eagle version="6.2">
+<eagle version="6.5.0">
 <drawing>
 <settings>
@@
 <wire x1="0" y1="198.12" x2="0" y2="0" width="0.1524" layer="94"/>
 <text x="48.26" y="190.5" size="3.81" layer="94">Raspberry PI connector</text>
-<text x="63.5" y="109.22" size="3.81" layer="94">2x CAN</text>
-<text x="149.86" y="157.48" size="3.81" layer="94">Optically isolated RS-485</text>
+<text x="63.5" y="109.22" size="3.81" layer="94">CAN</text>
+<text x="149.86" y="157.48" size="3.81" layer="94">RS-485 with Auto TX Enable</text>
 <text x="193.04" y="71.12" size="1.778" layer="94">Auto TX enable (40uS)</text>
 <wire x1="152.4" y1="0" x2="152.4" y2="27.94" width="0.1524" layer="94"/>
