File: stm32-board-adapter/stm32-board-adapter.sch (EAGLE design)
At the start: 35 parts, among them J2 22-05-7048-04, J3 22-05-7048-04, J4 22-05-7048-04, J5 22-05-7048-04

Commit message: stm32-board-adapter enhancements
Connections:
- net A1 renamed PA1_RTS2
- net A2 renamed PA2_TX2
- net B10 renamed B10_SCL2_TX3
- net B11 renamed B11_SDA2_RX3
- net MOSI2 renamed B15_MOSI2
- net SCK2 renamed B13_SCK2
- new net PA3_RX2: J3-4.S
- new net PA5_SCK1: J2-3.S
- net A3: no longer J3-4.S
- net SCK: no longer J2-3.S
Other:
- note added: "Adapter for Blue Pill board"
- note added: "CLK_DATA"
- note added: "CLK_DATA_2"
- note added: "I2C/UART"
- note added: "UART"
- note removed: "Adapter for STM32 board (LEDs)"
- moved on the sheet: J1, X1-1, X1-2
