File: cnc-controller/hardware/arduino-shield-label.brd (EAGLE design)
At the start: 253.6 x 20.3 mm, 0 parts

Commit message: cnc-controller mechanical
Other:
- board size 253.6 x 20.3 mm -> 94 x 53.3 mm
- board text added: "5V"
- board text added: "A0"
- board text added: "A1"
- board text added: "A2"
- board text added: "A3"
- board text added: "A4"
- board text added: "A5"
- board text added: "ABORT"
- board text added: "AUX"
- board text added: "Arduino / GRBL 1.1"
- board text added: "CNC Controller"
- board text added: "COOLANT"
- board text added: "D10"
- board text added: "D11"
- board text added: "D12"
- board text added: "D13"
- board text added: "D2"
- board text added: "D3"
- board text added: "D4"
- board text added: "D5"
- board text added: "D6"
- board text added: "D7"
- board text added: "D8"
- board text added: "D9"
- board text added: "DIR X"
- board text added: "DIR Y"
- board text added: "DIR Z"
- board text added: "GND"
- board text added: "HOLD"
- board text added: "LIMIT X"
- board text added: "LIMIT Y"
- board text added: "LIMIT Z"
- board text added: "PROBE"
- board text added: "RESUME"
- board text added: "RX"
- board text added: "SPINDLE DIR"
- board text added: "SPINDLE ENA"
- board text added: "SPINDLE PWM"
- board text added: "STEP X"
- board text added: "STEP Y"
- board text added: "STEP Z"
- board text added: "TX"
