File: breakout-ps2/breakout-ps2.kicad_pcb (KiCad board)
At the start: 2 copper layers, 20 x 12 mm, 12 parts, among them P1 MountingHole_Pad, P2 MountingHole_Pad, P3 MountingHole_Pad, P4 MountingHole_Pad, P5 MountingHole_Pad, P6 MountingHole_Pad

Commit message: breakout-ps2
Parts:
- moved C1 0.54 mm to (91.1, 97.5)
- moved C2 0.54 mm to (108.9, 97.5)
- moved C5 0.54 mm to (91.1, 102.5)
- moved C6 0.54 mm to (108.9, 102.5)
