File: triac-board/triac-board.kicad_pcb (KiCad board)
At the start: 2 copper layers, 100 x 80 mm, 24 parts, among them J1 Screw_Terminal_01x02, J2 Screw_Terminal_01x02, J3 Screw_Terminal_01x02, J4 Screw_Terminal_01x02, Q1 BTA16-600BW, Q2 BTA16-600BW, Q3 BTA16-600BW, Q4 BTA16-600BW, U1 MOC3063M, U2 MOC3063M, U3 MOC3063M, U4 MOC3063M

Commit message: triac-board
Parts:
- added J10: Screw_Terminal_01x02, TerminalBlock_Phoenix:TerminalBlock_Phoenix_MKDS-1,5-2_1x02_P5.00mm_Horizontal, F.Cu at (242.5, 136.0)
- added J11: Screw_Terminal_01x02, TerminalBlock_Phoenix:TerminalBlock_Phoenix_MKDS-1,5-2_1x02_P5.00mm_Horizontal, F.Cu at (242.5, 64.0)
- added J12: Screw_Terminal_01x02, TerminalBlock_Phoenix:TerminalBlock_Phoenix_MKDS-1,5-2_1x02_P5.00mm_Horizontal, F.Cu at (232.5, 64.0)
- added J13: Screw_Terminal_01x02, TerminalBlock_Phoenix:TerminalBlock_Phoenix_MKDS-1,5-2_1x02_P5.00mm_Horizontal, F.Cu at (222.5, 64.0)
- added J14: Screw_Terminal_01x02, TerminalBlock_Phoenix:TerminalBlock_Phoenix_MKDS-1,5-2_1x02_P5.00mm_Horizontal, F.Cu at (212.5, 64.0)
- added J15: Screw_Terminal_01x02, TerminalBlock_Phoenix:TerminalBlock_Phoenix_MKDS-1,5-2_1x02_P5.00mm_Horizontal, F.Cu at (202.5, 64.0)
- added J16: Screw_Terminal_01x02, TerminalBlock_Phoenix:TerminalBlock_Phoenix_MKDS-1,5-2_1x02_P5.00mm_Horizontal, F.Cu at (192.5, 64.0)
- added J17: Screw_Terminal_01x02, TerminalBlock_Phoenix:TerminalBlock_Phoenix_MKDS-1,5-2_1x02_P5.00mm_Horizontal, F.Cu at (182.5, 64.0)
- added J18: Screw_Terminal_01x02, TerminalBlock_Phoenix:TerminalBlock_Phoenix_MKDS-1,5-2_1x02_P5.00mm_Horizontal, F.Cu at (172.5, 64.0)
- added J19: Screw_Terminal_01x02, TerminalBlock_Phoenix:TerminalBlock_Phoenix_MKDS-1,5-2_1x02_P5.00mm_Horizontal, F.Cu at (162.5, 64.0)
- added J20: Conn_01x01_Male, Connector_Pin:Pin_D1.3mm_L11.0mm, F.Cu at (152.5, 64.0)
- added J21: Conn_01x01_Male, Connector_Pin:Pin_D1.3mm_L11.0mm, F.Cu at (247.5, 64.0)
- added J5: Screw_Terminal_01x02, TerminalBlock_Phoenix:TerminalBlock_Phoenix_MKDS-1,5-2_1x02_P5.00mm_Horizontal, F.Cu at (192.5, 136.0)
- added J6: Screw_Terminal_01x02, TerminalBlock_Phoenix:TerminalBlock_Phoenix_MKDS-1,5-2_1x02_P5.00mm_Horizontal, F.Cu at (202.5, 136.0)
- added J7: Screw_Terminal_01x02, TerminalBlock_Phoenix:TerminalBlock_Phoenix_MKDS-1,5-2_1x02_P5.00mm_Horizontal, F.Cu at (212.5, 136.0)
- added J8: Screw_Terminal_01x02, TerminalBlock_Phoenix:TerminalBlock_Phoenix_MKDS-1,5-2_1x02_P5.00mm_Horizontal, F.Cu at (222.5, 136.0)
- added J9: Screw_Terminal_01x02, TerminalBlock_Phoenix:TerminalBlock_Phoenix_MKDS-1,5-2_1x02_P5.00mm_Horizontal, F.Cu at (232.5, 136.0)
- added Q10: BTA16-600BW, triac-board:TO-220-3_Vertical_Staggered, F.Cu at (242.5, 110.0)
- added Q5: BTA16-600BW, triac-board:TO-220-3_Vertical_Staggered, F.Cu at (192.5, 110.0)
- added Q6: BTA16-600BW, triac-board:TO-220-3_Vertical_Staggered, F.Cu at (202.5, 110.0)
- added Q7: BTA16-600BW, triac-board:TO-220-3_Vertical_Staggered, F.Cu at (212.5, 110.0)
- added Q8: BTA16-600BW, triac-board:TO-220-3_Vertical_Staggered, F.Cu at (222.5, 110.0)
- added Q9: BTA16-600BW, triac-board:TO-220-3_Vertical_Staggered, F.Cu at (232.5, 110.0)
- added R10: 360 0.5W, Resistor_THT:R_Axial_DIN0309_L9.0mm_D3.2mm_P20.32mm_Horizontal, B.Cu at (245.0, 95.0)
- added R11: 1k2, Resistor_THT:R_Axial_DIN0207_L6.3mm_D2.5mm_P10.16mm_Horizontal, F.Cu at (157.5, 70.2)
- added R12: 1k2, Resistor_THT:R_Axial_DIN0207_L6.3mm_D2.5mm_P10.16mm_Horizontal, F.Cu at (169.5, 70.2)
- added R13: 1k2, Resistor_THT:R_Axial_DIN0207_L6.3mm_D2.5mm_P10.16mm_Horizontal, F.Cu at (177.5, 70.2)
- added R14: 1k2, Resistor_THT:R_Axial_DIN0207_L6.3mm_D2.5mm_P10.16mm_Horizontal, F.Cu at (187.5, 70.2)
- added R15: 1k2, Resistor_THT:R_Axial_DIN0207_L6.3mm_D2.5mm_P10.16mm_Horizontal, F.Cu at (197.5, 70.2)
- added R16: 1k2, Resistor_THT:R_Axial_DIN0207_L6.3mm_D2.5mm_P10.16mm_Horizontal, F.Cu at (207.5, 70.2)
- added R17: 1k2, Resistor_THT:R_Axial_DIN0207_L6.3mm_D2.5mm_P10.16mm_Horizontal, F.Cu at (217.5, 70.2)
- added R18: 1k2, Resistor_THT:R_Axial_DIN0207_L6.3mm_D2.5mm_P10.16mm_Horizontal, F.Cu at (227.5, 70.2)
- added R19: 1k2, Resistor_THT:R_Axial_DIN0207_L6.3mm_D2.5mm_P10.16mm_Horizontal, F.Cu at (240.5, 70.2)
- added R20: 1k2, Resistor_THT:R_Axial_DIN0207_L6.3mm_D2.5mm_P10.16mm_Horizontal, F.Cu at (247.5, 70.2)
- added R5: 360 0.5W, Resistor_THT:R_Axial_DIN0309_L9.0mm_D3.2mm_P20.32mm_Horizontal, B.Cu at (195.0, 95.0)
- added R6: 360 0.5W, Resistor_THT:R_Axial_DIN0309_L9.0mm_D3.2mm_P20.32mm_Horizontal, B.Cu at (205.0, 95.0)
- added R7: 360 0.5W, Resistor_THT:R_Axial_DIN0309_L9.0mm_D3.2mm_P20.32mm_Horizontal, B.Cu at (215.0, 95.0)
- added R8: 360 0.5W, Resistor_THT:R_Axial_DIN0309_L9.0mm_D3.2mm_P20.32mm_Horizontal, B.Cu at (225.0, 95.0)
- added R9: 360 0.5W, Resistor_THT:R_Axial_DIN0309_L9.0mm_D3.2mm_P20.32mm_Horizontal, B.Cu at (235.0, 95.0)
- added RV10: 275V, Varistor:RV_Disc_D9mm_W4.2mm_P5mm, F.Cu at (247.5, 120.0)
- added RV5: 275V, Varistor:RV_Disc_D9mm_W4.2mm_P5mm, F.Cu at (197.5, 120.0)
- added RV6: 275V, Varistor:RV_Disc_D9mm_W4.2mm_P5mm, F.Cu at (207.5, 120.0)
- added RV7: 275V, Varistor:RV_Disc_D9mm_W4.2mm_P5mm, F.Cu at (217.5, 120.0)
- added RV8: 275V, Varistor:RV_Disc_D9mm_W4.2mm_P5mm, F.Cu at (227.5, 120.0)
- added RV9: 275V, Varistor:RV_Disc_D9mm_W4.2mm_P5mm, F.Cu at (237.5, 120.0)
- added U10: MOC3063M, Package_DIP:DIP-6_W7.62mm, F.Cu at (247.5, 82.5)
- added U5: MOC3063M, Package_DIP:DIP-6_W7.62mm, F.Cu at (197.5, 82.5)
- added U6: MOC3063M, Package_DIP:DIP-6_W7.62mm, F.Cu at (207.5, 82.5)
- added U7: MOC3063M, Package_DIP:DIP-6_W7.62mm, F.Cu at (217.5, 82.5)
- added U8: MOC3063M, Package_DIP:DIP-6_W7.62mm, F.Cu at (227.5, 82.5)
- added U9: MOC3063M, Package_DIP:DIP-6_W7.62mm, F.Cu at (237.5, 82.5)
- Q2: value BTA16-600BW -> BTA16600BW
Connections:
- U1 pad 1: unconnected-(U1-Pad1) -> Net-(R11-Pad2)
- U1 pad 2: unconnected-(U1-Pad2) -> /IN1
- U2 pad 1: unconnected-(U2-Pad1) -> Net-(R12-Pad2)
- U2 pad 2: unconnected-(U2-Pad2) -> /IN2
- U3 pad 1: unconnected-(U3-Pad1) -> Net-(R13-Pad2)
- U3 pad 2: unconnected-(U3-Pad2) -> /IN3
- U4 pad 1: unconnected-(U4-Pad1) -> Net-(R14-Pad2)
- U4 pad 2: unconnected-(U4-Pad2) -> /IN4
Routing:
- net /VH_R: track 0.00 -> 51.2 mm
- net /VH_L: track 0.00 -> 51.2 mm
- net /IN1: track 0.00 -> 29.6 mm
- net Net-(J10-Pad1): track 0.00 -> 28.9 mm
- net /IN10: track 0.00 -> 28.3 mm
- net Net-(J9-Pad1): track 0.00 -> 28.1 mm
- net Net-(J8-Pad1): track 0.00 -> 27.2 mm
- net Net-(J7-Pad1): track 0.00 -> 27.2 mm
- net Net-(J6-Pad1): track 0.00 -> 27.2 mm
- net Net-(J5-Pad1): track 0.00 -> 27.2 mm
- net Net-(J9-Pad2): track 0.00 -> 26.6 mm
- net Net-(J10-Pad2): track 0.00 -> 25.8 mm
- net Net-(J8-Pad2): track 0.00 -> 24.9 mm
- net Net-(J7-Pad2): track 0.00 -> 24.5 mm
- net Net-(J6-Pad2): track 0.00 -> 24.5 mm
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Other:
- outline, holes or cut-outs redrawn
- board text added: "10x TRIAC BOARD"
- board text added: "2023"
- board text added: "230V HOT"
- board text added: "230V N"
- board text added: "Each channel"
- board text added: "GND L"
- board text added: "GND R"
- board text added: "HOT"
- board text added: "HOT terminal"
- board text added: "IN1"
- board text added: "IN10"
- board text added: "IN5"
- board text added: "IN6"
- board text added: "INSTALL HEATSINK"
- board text added: "ISOLATED TRIACS ONLY, SNUBBERLESS RECOMMENDED"
- board text added: "In that case, the board is connected with wires, soldered into R11-R20 terminals + GND R + GND L"
- board text added: "L,N"
- board text added: "L,N terminal"
- board text added: "LOAD"
- board text added: "MAX 100W"
- board text added: "QC:"
- board text added: "R11-R20 are installed only if there is no status/control daughterboard"
- board text added: "VH L"
- board text added: "VH R"
- board text added: "designed by"
- board text added: "semicontinuity"
- board text added: "v1.0"

Commit message: triac-board
Parts:
- added U1 (x3): MOC3063M, Package_DIP:DIP-6_W7.62mm, F.Cu at (156.1, 82.5)
- moved U1 1.44 mm to (156.1, 82.5)
- moved R1 1.23 mm to (154.3, 94.0)
- moved R10 1.23 mm to (245.7, 94.0)
- moved R2 1.15 mm to (164.4, 94.0)
- moved R9 1.15 mm to (235.6, 94.0)
- moved R3 1.12 mm to (174.5, 94.0)
- moved R8 1.08 mm to (225.4, 94.0)
- moved R4 1.03 mm to (184.8, 94.0)
- moved R7 1.03 mm to (215.2, 94.0)
- moved R5 1.00 mm to (194.9, 94.0)
- moved R6 1.00 mm to (205.1, 94.0)
- moved RV1 0.90 mm to (156.6, 120.0)
- moved RV10 0.90 mm to (248.4, 120.0)
- moved J1 0.72 mm to (151.8, 136.0)
- moved J10 0.72 mm to (243.2, 136.0)
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Routing:
- net Net-(J1-Pad2): track 26.6 -> 24.5 mm
- net Net-(J1-Pad1): track 28.5 -> 27.1 mm
- net Net-(J2-Pad2): track 25.3 -> 26.7 mm
- net Net-(J10-Pad1): track 28.9 -> 27.6 mm
- net Net-(J2-Pad1): track 29.3 -> 28.1 mm
- net Net-(J10-Pad2): track 25.8 -> 24.7 mm
- net Net-(Q2-Pad3): track 24.0 -> 23.0 mm
- net Net-(R9-Pad1): track 5.92 -> 4.92 mm
- net Net-(R8-Pad1): track 5.92 -> 4.92 mm
- net Net-(R7-Pad1): track 5.92 -> 4.92 mm
- net Net-(R6-Pad1): track 5.92 -> 4.92 mm
- net Net-(R5-Pad1): track 5.92 -> 4.92 mm
- net Net-(R4-Pad1): track 5.92 -> 4.92 mm
- net Net-(R2-Pad1): track 5.92 -> 4.92 mm
- net Net-(R10-Pad1): track 5.92 -> 4.92 mm
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Other:
- outline, holes or cut-outs redrawn
- board text added: "5.00"
- board text added: "5.08"
- board text added: "ISOLATED TRIACS ONLY, SNUBBERLESS RECOMMENDED (BTA16-600BW)"
- board text removed: "ISOLATED TRIACS ONLY, SNUBBERLESS RECOMMENDED"

Commit message: triac-board
Parts:
- removed the U1 at (156.1, 82.5) (x3)
- added D1: LED, LED_THT:LED_D3.0mm, F.Cu at (155.0, 46.6)
- added D10: LED, LED_THT:LED_D3.0mm, F.Cu at (245.0, 46.6)
- added D2: LED, LED_THT:LED_D3.0mm, F.Cu at (165.0, 46.6)
- added D3: LED, LED_THT:LED_D3.0mm, F.Cu at (175.0, 46.6)
- added D4: LED, LED_THT:LED_D3.0mm, F.Cu at (185.0, 46.6)
- added D5: LED, LED_THT:LED_D3.0mm, F.Cu at (195.0, 46.6)
- added D6: LED, LED_THT:LED_D3.0mm, F.Cu at (205.0, 46.6)
- added D7: LED, LED_THT:LED_D3.0mm, F.Cu at (215.0, 46.6)
- added D8: LED, LED_THT:LED_D3.0mm, F.Cu at (225.0, 46.6)
- added D9: LED, LED_THT:LED_D3.0mm, F.Cu at (235.0, 46.6)
- added I1: Conn_01x01_Female, Connector_Wire:SolderWire-0.5sqmm_1x01_D0.9mm_OD2.3mm, F.Cu at (158.5, 49.5)
- added I10: Conn_01x01_Female, Connector_Wire:SolderWire-0.5sqmm_1x01_D0.9mm_OD2.3mm, F.Cu at (248.5, 49.5)
- added I2: Conn_01x01_Female, Connector_Wire:SolderWire-0.5sqmm_1x01_D0.9mm_OD2.3mm, F.Cu at (168.5, 49.5)
- added I3: Conn_01x01_Female, Connector_Wire:SolderWire-0.5sqmm_1x01_D0.9mm_OD2.3mm, F.Cu at (178.5, 49.5)
- added I4: Conn_01x01_Female, Connector_Wire:SolderWire-0.5sqmm_1x01_D0.9mm_OD2.3mm, F.Cu at (188.5, 49.5)
- added I5: Conn_01x01_Female, Connector_Wire:SolderWire-0.5sqmm_1x01_D0.9mm_OD2.3mm, F.Cu at (198.5, 49.5)
- added I6: Conn_01x01_Female, Connector_Wire:SolderWire-0.5sqmm_1x01_D0.9mm_OD2.3mm, F.Cu at (208.5, 49.5)
- added I7: Conn_01x01_Female, Connector_Wire:SolderWire-0.5sqmm_1x01_D0.9mm_OD2.3mm, F.Cu at (218.5, 49.5)
- added I8: Conn_01x01_Female, Connector_Wire:SolderWire-0.5sqmm_1x01_D0.9mm_OD2.3mm, F.Cu at (228.5, 49.5)
- added I9: Conn_01x01_Female, Connector_Wire:SolderWire-0.5sqmm_1x01_D0.9mm_OD2.3mm, F.Cu at (238.5, 49.5)
- added J22: Conn_01x01_Female, Connector_Wire:SolderWire-0.5sqmm_1x01_D0.9mm_OD2.3mm, F.Cu at (198.5, 56.5)
- added J23: Conn_01x01_Female, Connector_Wire:SolderWire-0.5sqmm_1x01_D0.9mm_OD2.3mm, F.Cu at (158.5, 56.5)
- added J24: Conn_01x01_Female, Connector_Wire:SolderWire-0.5sqmm_1x01_D0.9mm_OD2.3mm, F.Cu at (208.5, 56.5)
- added J25: Conn_01x01_Female, Connector_Wire:SolderWire-0.5sqmm_1x01_D0.9mm_OD2.3mm, F.Cu at (218.5, 56.5)
- added J26: Conn_01x01_Female, Connector_Wire:SolderWire-0.5sqmm_1x01_D0.9mm_OD2.3mm, F.Cu at (168.5, 56.5)
- added J27: Conn_01x01_Female, Connector_Wire:SolderWire-0.5sqmm_1x01_D0.9mm_OD2.3mm, F.Cu at (228.5, 56.5)
- added J28: Conn_01x01_Female, Connector_Wire:SolderWire-0.5sqmm_1x01_D0.9mm_OD2.3mm, F.Cu at (238.5, 56.5)
- added J29: Conn_01x01_Female, Connector_Wire:SolderWire-0.5sqmm_1x01_D0.9mm_OD2.3mm, F.Cu at (178.5, 56.5)
- added J30: Conn_01x01_Female, Connector_Wire:SolderWire-0.5sqmm_1x01_D0.9mm_OD2.3mm, F.Cu at (248.5, 56.5)
- added J31: Conn_01x01_Male, Connector_Pin:Pin_D1.3mm_L11.0mm, F.Cu at (197.5, 74.0)
- added J32: Conn_01x01_Female, Connector_Wire:SolderWire-0.5sqmm_1x01_D0.9mm_OD2.3mm, F.Cu at (188.5, 56.5)
- added J33: Conn_01x01_Male, Connector_Pin:Pin_D1.3mm_L11.0mm, F.Cu at (202.5, 74.0)
- added J34: Conn_01x01_Male, Connector_Pin:Pin_D1.3mm_L11.0mm, F.Cu at (197.5, 77.7)
- added J35: Conn_01x01_Male, Connector_Pin:Pin_D1.3mm_L11.0mm, F.Cu at (202.5, 77.7)
- added OC1: Conn_01x01_Female, Connector_Wire:SolderWire-0.5sqmm_1x01_D0.9mm_OD2.3mm, F.Cu at (151.5, 54.3)
- added OC10: Conn_01x01_Female, Connector_Wire:SolderWire-0.5sqmm_1x01_D0.9mm_OD2.3mm, F.Cu at (241.5, 54.2)
- added OC2: Conn_01x01_Female, Connector_Wire:SolderWire-0.5sqmm_1x01_D0.9mm_OD2.3mm, F.Cu at (161.5, 54.2)
- added OC3: Conn_01x01_Female, Connector_Wire:SolderWire-0.5sqmm_1x01_D0.9mm_OD2.3mm, F.Cu at (171.5, 54.2)
- added OC4: Conn_01x01_Female, Connector_Wire:SolderWire-0.5sqmm_1x01_D0.9mm_OD2.3mm, F.Cu at (181.5, 54.2)
- added OC5: Conn_01x01_Female, Connector_Wire:SolderWire-0.5sqmm_1x01_D0.9mm_OD2.3mm, F.Cu at (191.5, 54.2)
- added OC6: Conn_01x01_Female, Connector_Wire:SolderWire-0.5sqmm_1x01_D0.9mm_OD2.3mm, F.Cu at (201.5, 54.2)
- added OC7: Conn_01x01_Female, Connector_Wire:SolderWire-0.5sqmm_1x01_D0.9mm_OD2.3mm, F.Cu at (211.5, 54.2)
- added OC8: Conn_01x01_Female, Connector_Wire:SolderWire-0.5sqmm_1x01_D0.9mm_OD2.3mm, F.Cu at (221.5, 54.2)
- added OC9: Conn_01x01_Female, Connector_Wire:SolderWire-0.5sqmm_1x01_D0.9mm_OD2.3mm, F.Cu at (231.5, 54.2)
- added R21: 1k2, Resistor_THT:R_Axial_DIN0207_L6.3mm_D2.5mm_P7.62mm_Horizontal, F.Cu at (151.5, 51.8)
- added R22: 1k2, Resistor_THT:R_Axial_DIN0207_L6.3mm_D2.5mm_P7.62mm_Horizontal, F.Cu at (161.5, 51.8)
- added R23: 1k2, Resistor_THT:R_Axial_DIN0207_L6.3mm_D2.5mm_P7.62mm_Horizontal, F.Cu at (171.5, 51.8)
- added R24: 1k2, Resistor_THT:R_Axial_DIN0207_L6.3mm_D2.5mm_P7.62mm_Horizontal, F.Cu at (181.5, 51.8)
- added R25: 1k2, Resistor_THT:R_Axial_DIN0207_L6.3mm_D2.5mm_P7.62mm_Horizontal, F.Cu at (191.5, 51.8)
- added R26: 1k2, Resistor_THT:R_Axial_DIN0207_L6.3mm_D2.5mm_P7.62mm_Horizontal, F.Cu at (201.5, 51.8)
- added R27: 1k2, Resistor_THT:R_Axial_DIN0207_L6.3mm_D2.5mm_P7.62mm_Horizontal, F.Cu at (211.5, 51.8)
- added R28: 1k2, Resistor_THT:R_Axial_DIN0207_L6.3mm_D2.5mm_P7.62mm_Horizontal, F.Cu at (221.5, 51.8)
- added R29: 1k2, Resistor_THT:R_Axial_DIN0207_L6.3mm_D2.5mm_P7.62mm_Horizontal, F.Cu at (231.5, 51.8)
- added R30: 1k2, Resistor_THT:R_Axial_DIN0207_L6.3mm_D2.5mm_P7.62mm_Horizontal, F.Cu at (241.5, 51.8)
- added SW1: SW_SPDT, Connector_PinHeader_2.54mm:PinHeader_1x03_P2.54mm_Vertical, F.Cu at (155.0, 49.5)
- added SW10: SW_SPDT, Connector_PinHeader_2.54mm:PinHeader_1x03_P2.54mm_Vertical, F.Cu at (245.0, 49.5)
- added SW2: SW_SPDT, Connector_PinHeader_2.54mm:PinHeader_1x03_P2.54mm_Vertical, F.Cu at (165.0, 49.5)
- added SW3: SW_SPDT, Connector_PinHeader_2.54mm:PinHeader_1x03_P2.54mm_Vertical, F.Cu at (175.0, 49.5)
- added SW4: SW_SPDT, Connector_PinHeader_2.54mm:PinHeader_1x03_P2.54mm_Vertical, F.Cu at (185.0, 49.5)
- added SW5: SW_SPDT, Connector_PinHeader_2.54mm:PinHeader_1x03_P2.54mm_Vertical, F.Cu at (195.0, 49.5)
- added SW6: SW_SPDT, Connector_PinHeader_2.54mm:PinHeader_1x03_P2.54mm_Vertical, F.Cu at (205.0, 49.5)
- added SW7: SW_SPDT, Connector_PinHeader_2.54mm:PinHeader_1x03_P2.54mm_Vertical, F.Cu at (215.0, 49.5)
- added SW8: SW_SPDT, Connector_PinHeader_2.54mm:PinHeader_1x03_P2.54mm_Vertical, F.Cu at (225.0, 49.5)
- added SW9: SW_SPDT, Connector_PinHeader_2.54mm:PinHeader_1x03_P2.54mm_Vertical, F.Cu at (235.0, 49.5)
- Q2: value BTA16600BW -> BTA16-600BW
- moved R19 10.5 mm to (230.0, 70.2)
- moved R15 5.04 mm to (192.5, 70.2)
- moved R18 4.70 mm to (222.8, 70.2)
- moved R11 4.00 mm to (153.5, 70.2)
- moved R14 2.50 mm to (185.0, 70.2)
- moved R17 2.30 mm to (215.2, 70.2)
- moved R20 1.90 mm to (245.6, 70.2)
- moved Q1 1.00 mm to (151.8, 111.0)
- moved Q10 1.00 mm to (243.2, 111.0)
- moved Q2 1.00 mm to (161.9, 111.0)
- moved Q3 1.00 mm to (172.1, 111.0)
- moved Q4 1.00 mm to (182.3, 111.0)
- moved Q5 1.00 mm to (192.4, 111.0)
- moved Q6 1.00 mm to (202.6, 111.0)
- moved Q7 1.00 mm to (212.7, 111.0)
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Connections:
- R11 pad 1: /VH_L -> /IN1
- R12 pad 1: /VH_L -> /IN2
- R13 pad 1: /VH_L -> /IN3
- R14 pad 1: /VH_L -> /IN4
- R15 pad 1: /VH_L -> /IN5
- R16 pad 1: /VH_R -> /IN6
- R17 pad 1: /VH_R -> /IN7
- R18 pad 1: /VH_R -> /IN8
- R19 pad 1: /VH_R -> /IN9
- R20 pad 1: /VH_R -> /IN10
- U1 pad 1: Net-(R11-Pad2) -> /VHL
- U1 pad 2: /IN1 -> Net-(R11-Pad2)
- U10 pad 1: Net-(R20-Pad2) -> /VHR
- U10 pad 2: /IN10 -> Net-(R20-Pad2)
- U2 pad 1: Net-(R12-Pad2) -> /VHL
- U2 pad 2: /IN2 -> Net-(R12-Pad2)
- U3 pad 1: Net-(R13-Pad2) -> /VHL
- U3 pad 2: /IN3 -> Net-(R13-Pad2)
- U4 pad 1: Net-(R14-Pad2) -> /VHL
- U4 pad 2: /IN4 -> Net-(R14-Pad2)
- U5 pad 1: Net-(R15-Pad2) -> /VHL
- U5 pad 2: /IN5 -> Net-(R15-Pad2)
- U6 pad 1: Net-(R16-Pad2) -> /VHR
- U6 pad 2: /IN6 -> Net-(R16-Pad2)
- U7 pad 1: Net-(R17-Pad2) -> /VHR
- U7 pad 2: /IN7 -> Net-(R17-Pad2)
- U8 pad 1: Net-(R18-Pad2) -> /VHR
- U8 pad 2: /IN8 -> Net-(R18-Pad2)
- U9 pad 1: Net-(R19-Pad2) -> /VHR
- U9 pad 2: /IN9 -> Net-(R19-Pad2)
Routing:
- net /VHR: track 0.00 -> 115.9 mm
- net /VHL: track 0.00 -> 108.6 mm
- net /GND_L: track 10.0 -> 81.5 mm
- net /GND_R: track 10.0 -> 75.8 mm
- net /VH_L: track 51.2 -> 23.5 mm
- net /VH_R: track 51.2 -> 23.6 mm
- net /IN2: track 21.9 -> 7.29 mm
- net /IN9: track 21.8 -> 7.29 mm
- net /IN3: track 19.7 -> 6.25 mm
- net /IN5: track 21.6 -> 8.30 mm
- net /IN8: track 19.7 -> 6.37 mm
- net /IN6: track 21.6 -> 8.30 mm
- net /IN10: track 28.9 -> 15.7 mm
- net /IN7: track 19.7 -> 7.20 mm
- net /IN4: track 19.5 -> 7.29 mm
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Other:
- board size 100 x 80 mm -> 100 x 97 mm
- board text added: "..."
- board text added: "INPUTS ACTIVE LOW"
- board text added: "TERM FUSES"
- board text added: "VH, VR = +24V"
- board text added: "VL"
- board text added: "VR"
- board text added: "X1"
- board text added: "X10"
- board text added: "X5"
- board text added: "X6"
- board text added: "Y1"
- board text added: "Y10"
- board text added: "Y2"
- board text added: "Y3"
- board text added: "Y4"
- board text added: "Y5"
- board text added: "Y6"
- board text added: "Y7"
- board text added: "Y8"
- board text added: "Y9"
- board text removed: "IN1"
- board text removed: "IN10"
- board text removed: "IN5"
- board text removed: "IN6"
- board text removed: "In that case, the board is connected with wires, soldered into R11-R20 terminals + GND R + GND L"
- board text removed: "R11-R20 are installed only if there is no status/control daughterboard"
- board text removed: "VH L"
- board text removed: "VH R"
