File: triac-board/triac-board.kicad_sch (KiCad schematic)
At the start: 24 parts, among them J1 Screw_Terminal_01x02, J2 Screw_Terminal_01x02, J3 Screw_Terminal_01x02, J4 Screw_Terminal_01x02, Q1 BTA16-600BW, Q2 BTA16-600BW, Q3 BTA16-600BW, Q4 BTA16-600BW, U1 MOC3063M, U2 MOC3063M, U3 MOC3063M, U4 MOC3063M

Commit message: triac-board
Parts:
- added J10, J11, J12, J13, J14, J15, J16, J17, J18, J19, J5, J6, J7, J8, J9: Screw_Terminal_01x02, TerminalBlock_Phoenix:TerminalBlock_Phoenix_MKDS-1,5-2_1x02_P5.00mm_Horizontal, symbol Connector:Screw_Terminal_01x02
- added J20, J21: Conn_01x01_Male, Connector_Pin:Pin_D1.3mm_L11.0mm, symbol Connector:Conn_01x01_Male
- added Q10, Q5, Q6, Q7, Q8, Q9: BTA16-600BW, triac-board:TO-220-3_Vertical_Staggered, symbol Triac_Thyristor:BTA16-600BW
- added R10, R5, R6, R7, R8, R9: 360 0.5W, Resistor_THT:R_Axial_DIN0309_L9.0mm_D3.2mm_P20.32mm_Horizontal, symbol Device:R
- added R11, R12, R13, R14, R15, R16, R17, R18, R19, R20: 1k2, Resistor_THT:R_Axial_DIN0207_L6.3mm_D2.5mm_P10.16mm_Horizontal, symbol Device:R
- added RV10, RV5, RV6, RV7, RV8, RV9: 275V, Varistor:RV_Disc_D9mm_W4.2mm_P5mm, symbol Device:Varistor
- added U10, U5, U6, U7, U8, U9: MOC3063M, Package_DIP:DIP-6_W7.62mm, symbol Relay_SolidState:MOC3063M
Connections:
- net at U1.1: now also R11.2
- net IN1: now reaches U1.2
- net IN1: now also J18.2 (Pin_2)
- net at U2.1: now also R12.2
- net IN2: now reaches U2.2
- net IN2: now also J18.1 (Pin_1)
- net at U3.1: now also R13.2
- net IN3: now reaches U3.2
- net IN3: now also J17.2 (Pin_2)
- net at U4.1: now also R14.2
- net IN4: now reaches U4.2
- net IN4: now also J17.1 (Pin_1)
- new net: J7.2 (Pin_2), Q7.2 (A2), R7.2, RV7.1
- new net: J7.1 (Pin_1), Q7.1 (A1), RV7.2
- new net: R18.2, U8.1
- new net: Q8.3 (G), U8.4
- new net: R8.1, U8.6
- new net: J9.1 (Pin_1), Q9.1 (A1), RV9.2
- new net: J9.2 (Pin_2), Q9.2 (A2), R9.2, RV9.1
- new net: Q9.3 (G), U9.4
- new net: R5.1, U5.6
- new net: J5.2 (Pin_2), Q5.2 (A2), R5.2, RV5.1
- new net: R15.2, U5.1
- new net: Q7.3 (G), U7.4
- new net: J5.1 (Pin_1), Q5.1 (A1), RV5.2
- new net: R19.2, U9.1
- new net: R9.1, U9.6
- new net: J8.1 (Pin_1), Q8.1 (A1), RV8.2
- new net: J8.2 (Pin_2), Q8.2 (A2), R8.2, RV8.1
- new net: R16.2, U6.1
- new net: R20.2, U10.1
- new net: R7.1, U7.6
- new net: Q6.3 (G), U6.4
- new net: R6.1, U6.6
- new net: J6.1 (Pin_1), Q6.1 (A1), RV6.2
- new net: J6.2 (Pin_2), Q6.2 (A2), R6.2, RV6.1
- new net: J10.1 (Pin_1), Q10.1 (A1), RV10.2
- new net: J10.2 (Pin_2), Q10.2 (A2), R10.2, RV10.1
- new net: Q10.3 (G), U10.4
- new net: R10.1, U10.6
- new net: R17.2, U7.1
- new net: Q5.3 (G), U5.4
- new net GND_L: J19.1 (Pin_1), J19.2 (Pin_2), J20.1 (Pin_1)
- new net GND_R: J11.1 (Pin_1), J11.2 (Pin_2), J21.1 (Pin_1)
- new net IN10: J12.1 (Pin_1), U10.2
- new net IN5: J16.2 (Pin_2), U5.2
- new net IN6: J14.1 (Pin_1), U6.2
- new net IN7: J13.2 (Pin_2), U7.2
- new net IN8: J13.1 (Pin_1), U8.2
- new net IN9: J12.2 (Pin_2), U9.2
- new net VH_L: J15.2 (Pin_2), J16.1 (Pin_1), R11.1, R12.1, R13.1, R14.1, R15.1
- new net VH_R: J14.2 (Pin_2), J15.1 (Pin_1), R16.1, R17.1, R18.1, R19.1, R20.1
Other:
- moved on the sheet: J1, J2, J3, J4, Q1, Q2, Q3, Q4, R1, R2, R3, R4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

Commit message: triac-board
Parts:
- added D1, D10, D2, D3, D4, D5, D6, D7, D8, D9: LED, LED_THT:LED_D3.0mm, symbol Device:LED
- added I1, I10, I2, I3, I4, I5, I6, I7, I8, I9, J22, J23, J24, J25, J26, J27, J28, J29, J30, J32, OC1, OC10, OC2, OC3, OC4, OC5, OC6, OC7, OC8, OC9: Conn_01x01_Female, Connector_Wire:SolderWire-0.5sqmm_1x01_D0.9mm_OD2.3mm, symbol Connector:Conn_01x01_Female
- added J31, J33, J34, J35: Conn_01x01_Male, Connector_Pin:Pin_D1.3mm_L11.0mm, symbol Connector:Conn_01x01_Male
- added R21, R22, R23, R24, R25, R26, R27, R28, R29, R30: 1k2, Resistor_THT:R_Axial_DIN0207_L6.3mm_D2.5mm_P7.62mm_Horizontal, symbol Device:R
- added SW1, SW10, SW2, SW3, SW4, SW5, SW6, SW7, SW8, SW9: SW_SPDT, Connector_PinHeader_2.54mm:PinHeader_1x03_P2.54mm_Vertical, symbol Switch:SW_SPDT
Connections:
- net GND_L: now also J22.1 (Pin_1), J23.1 (Pin_1), J26.1 (Pin_1), J29.1 (Pin_1), J32.1 (Pin_1), SW1.3 (C), SW2.3 (C), SW3.3 (C), SW4.3 (C), SW5.3 (C)
- net GND_R: now also J24.1 (Pin_1), J25.1 (Pin_1), J27.1 (Pin_1), J28.1 (Pin_1), J30.1 (Pin_1), SW10.3 (C), SW6.3 (C), SW7.3 (C), SW8.3 (C), SW9.3 (C)
- net IN1: now also R11.1; no longer U1.2
- net IN10: now also R20.1; no longer U10.2
- net IN2: now also R12.1; no longer U2.2
- net IN3: now also R13.1; no longer U3.2
- net IN4: now also R14.1; no longer U4.2
- net IN5: now also R15.1; no longer U5.2
- net IN6: now also R16.1; no longer U6.2
- net IN7: now also R17.1; no longer U7.2
- net IN8: now also R18.1; no longer U8.2
- net IN9: now also R19.1; no longer U9.2
- net VH_L: now also J31.1 (Pin_1); no longer R11.1, R12.1, R13.1, R14.1, R15.1
- net VH_R: now also J33.1 (Pin_1); no longer R16.1, R17.1, R18.1, R19.1, R20.1
- net at R18.2: now also U8.2; no longer U8.1
- net at R11.2: now also U1.2; no longer U1.1
- net at R15.2: now also U5.2; no longer U5.1
- net at R19.2: now also U9.2; no longer U9.1
- net at R16.2: now also U6.2; no longer U6.1
- net at R13.2: now also U3.2; no longer U3.1
- net at R12.2: now also U2.2; no longer U2.1
- net at R20.2: now also U10.2; no longer U10.1
- net at R14.2: now also U4.2; no longer U4.1
- net at R17.2: now also U7.2; no longer U7.1
- new net: OC7.1 (Pin_1), R27.1
- new net: D7.2 (A), R27.2
- new net: OC2.1 (Pin_1), R22.1
- new net: D2.2 (A), R22.2
- new net: OC4.1 (Pin_1), R24.1
- new net: D4.2 (A), R24.2
- new net: OC10.1 (Pin_1), R30.1
- new net: D10.2 (A), R30.2
- new net: OC6.1 (Pin_1), R26.1
- new net: D6.2 (A), R26.2
- new net: OC9.1 (Pin_1), R29.1
- new net: D9.2 (A), R29.2
- new net: OC1.1 (Pin_1), R21.1
- new net: OC5.1 (Pin_1), R25.1
- new net: D5.2 (A), R25.2
- new net: D8.2 (A), R28.2
- new net: OC3.1 (Pin_1), R23.1
- new net: D1.2 (A), R21.2
- new net: OC8.1 (Pin_1), R28.1
- new net: D3.2 (A), R23.2
- new net I1: D1.1 (K), I1.1 (Pin_1), SW1.1 (A), SW1.2 (B)
- new net I10: D10.1 (K), I10.1 (Pin_1), SW10.1 (A), SW10.2 (B)
- new net I2: D2.1 (K), I2.1 (Pin_1), SW2.1 (A), SW2.2 (B)
- new net I3: D3.1 (K), I3.1 (Pin_1), SW3.1 (A), SW3.2 (B)
- new net I4: D4.1 (K), I4.1 (Pin_1), SW4.1 (A), SW4.2 (B)
- new net I5: D5.1 (K), I5.1 (Pin_1), SW5.1 (A), SW5.2 (B)
- new net I6: D6.1 (K), I6.1 (Pin_1), SW6.1 (A), SW6.2 (B)
- new net I7: D7.1 (K), I7.1 (Pin_1), SW7.1 (A), SW7.2 (B)
- new net I8: D8.1 (K), I8.1 (Pin_1), SW8.1 (A), SW8.2 (B)
- new net I9: D9.1 (K), I9.1 (Pin_1), SW9.1 (A), SW9.2 (B)
- new net VHL: J34.1 (Pin_1), U1.1, U2.1, U3.1, U4.1, U5.1
- new net VHR: J35.1 (Pin_1), U10.1, U6.1, U7.1, U8.1, U9.1
Other:
- note added: "10x TRIAC BOARD"
- moved on the sheet: H1, H2, H3, H4, J1, J10, J11, J12, J13, J14, J15, J16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
