File: din-3u-button-panel/din-3u-button-panel.kicad_pcb (KiCad board)
At the start: 2 copper layers, 64 x 84 mm, 10 parts, among them J1 Screw_Terminal_01x02, J10 AUX_INS, J2 Screw_Terminal_01x02, J3 Screw_Terminal_01x02, J4 Screw_Terminal_01x02, J5 Screw_Terminal_01x02, J6 V_ST_HWS, J7 V_ST_CWS, J8 W_CT_HWS, J9 W_CT_CWS

Commit message: din-3u-button-panel: update
Parts:
- moved J10 145.1 mm to (122.8, 62.0), turned to 180 degrees
- moved J9 129.6 mm to (112.7, 62.0), turned to 180 degrees
- moved J8 114.0 mm to (102.5, 62.0), turned to 180 degrees
- moved J5 101.7 mm to (117.8, 138.0)
- moved J7 98.5 mm to (92.3, 62.0), turned to 180 degrees
- moved J4 87.9 mm to (107.7, 138.0)
- moved J3 74.8 mm to (97.5, 138.0)
Changed lines of the file:
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@@
         (effects (font (size 1 1) (thickness 0.15)))
     )
-    (fp_text value "V_ST_HWS" (at 2.54 5.66) (layer "F.Fab")
+    (fp_text value "V_ST_HWS" (at 2.54 5.66) (layer "F.Fab") hide
         (effects (font (size 1 1) (thickness 0.15)))
     )
@@
   )
   (footprint "TerminalBlock_Phoenix:TerminalBlock_Phoenix_MKDS-1,5-2-5.08_1x02_P5.08mm_Horizontal" (layer "F.Cu")
-    (at 24.7 179)
+    (at 117.82 138)
     (descr "Terminal Block Phoenix MKDS-1,5-2-5.08, 2 pins, pitch 5.08mm, size 10.2x9.8mm^2, drill diamater 1.3mm, pad diameter 2.6mm, see http://www.farnell.com/datasheets/100425.pdf, script-generated using https://github.com/pointhi/kicad-footprint-generator/scripts/TerminalBlock_Phoenix")
     (tags "THT Terminal Block Phoenix MKDS-1,5-2-5.08 pitch 5.08mm size 10.2x9.8mm^2 drill 1.3mm pad 2.6mm")
@@
         (effects (font (size 1 1) (thickness 0.15)))
     )
-    (fp_text value "Screw_Terminal_01x02" (at 2.54 5.66) (layer "F.Fab")
+    (fp_text value "Screw_Terminal_01x02" (at 2.54 5.66) (layer "F.Fab") hide
         (effects (font (size 1 1) (thickness 0.15)))
     )
@@
   )
   (footprint "TerminalBlock_Phoenix:TerminalBlock_Phoenix_MKDS-1,5-2-5.08_1x02_P5.08mm_Horizontal" (layer "F.Cu")
-    (at 24.7 155.28)
+    (at 97.5 138)
     (descr "Terminal Block Phoenix MKDS-1,5-2-5.08, 2 pins, pitch 5.08mm, size 10.2x9.8mm^2, drill diamater 1.3mm, pad diameter 2.6mm, see http://www.farnell.com/datasheets/100425.pdf, script-generated using https://github.com/pointhi/kicad-footprint-generator/scripts/TerminalBlock_Phoenix")
     (tags "THT Terminal Block Phoenix MKDS-1,5-2-5.08 pitch 5.08mm size 10.2x9.8mm^2 drill 1.3mm pad 2.6mm")
@@
         (effects (font (size 1 1) (thickness 0.15)))
     )
-    (fp_text value "Screw_Terminal_01x02" (at 2.54 5.66) (layer "F.Fab")
+    (fp_text value "Screw_Terminal_01x02" (at 2.54 5.66) (layer "F.Fab") hide
         (effects (font (size 1 1) (thickness 0.15)))
     )
@@
   )
   (footprint "TerminalBlock_Phoenix:TerminalBlock_Phoenix_MKDS-1,5-2-5.08_1x02_P5.08mm_Horizontal" (layer "F.Cu")
-    (at 36.92 167.14)
+    (at 112.66 62 180)
     (descr "Terminal Block Phoenix MKDS-1,5-2-5.08, 2 pins, pitch 5.08mm, size 10.2x9.8mm^2, drill diamater 1.3mm, pad diameter 2.6mm, see http://www.farnell.com/datasheets/100425.pdf, script-generated using https://github.com/pointhi/kicad-footprint-generator/scripts/TerminalBlock_Phoenix")
     (tags "THT Terminal Block Phoenix MKDS-1,5-2-5.08 pitch 5.08mm size 10.2x9.8mm^2 drill 1.3mm pad 2.6mm")
@@
         (effects (font (size 1 1) (thickness 0.15)))
     )
-    (fp_text value "W_CT_CWS" (at 2.54 5.66) (layer "F.Fab")
+    (fp_text value "W_CT_CWS" (at 2.54 5.66) (layer "F.Fab") hide
         (effects (font (size 1 1) (thickness 0.15)))
     )
@@
     (fp_circle (center 5.08 0) (end 6.58 0)
       (stroke (width 0.1) (type solid)) (fill none) (layer "F.Fab"))
-    (pad "1" thru_hole rect (at 0 0) (size 2.6 2.6) (drill 1.3) (layers "*.Cu" "*.Mask")
+    (pad "1" thru_hole rect (at 0 0 180) (size 2.6 2.6) (drill 1.3) (layers "*.Cu" "*.Mask")
       (net 13 "/X7") (pinfunction "Pin_1") (pintype "passive"))
-    (pad "2" thru_hole circle (at 5.08 0) (size 2.6 2.6) (drill 1.3) (layers "*.Cu" "*.Mask")
+    (pad "2" thru_hole circle (at 5.08 0 180) (size 2.6 2.6) (drill 1.3) (layers "*.Cu" "*.Mask")
       (net 14 "/X6") (pinfunction "Pin_2") (pintype "passive"))
     (model "${KICAD6_3DMODEL_DIR}/TerminalBlock_Phoenix.3dshapes/TerminalBlock_Phoenix_MKDS-1,5-2-5.08_1x02_P5.08mm_Horizontal.wrl"
@@
   )
   (footprint "TerminalBlock_Phoenix:TerminalBlock_Phoenix_MKDS-1,5-2-5.08_1x02_P5.08mm_Horizontal" (layer "F.Cu")
-    (at 36.92 179)
+    (at 122.82 62 180)
     (descr "Terminal Block Phoenix MKDS-1,5-2-5.08, 2 pins, pitch 5.08mm, size 10.2x9.8mm^2, drill diamater 1.3mm, pad diameter 2.6mm, see http://www.farnell.com/datasheets/100425.pdf, script-generated using https://github.com/pointhi/kicad-footprint-generator/scripts/TerminalBlock_Phoenix")
     (tags "THT Terminal Block Phoenix MKDS-1,5-2-5.08 pitch 5.08mm size 10.2x9.8mm^2 drill 1.3mm pad 2.6mm")
@@
         (effects (font (size 1 1) (thickness 0.15)))
     )
-    (fp_text value "AUX_INS" (at 2.54 5.66) (layer "F.Fab")
+    (fp_text value "AUX_INS" (at 2.54 5.66) (layer "F.Fab") hide
         (effects (font (size 1 1) (thickness 0.15)))
     )
@@
     (fp_circle (center 5.08 0) (end 6.58 0)
       (stroke (width 0.1) (type solid)) (fill none) (layer "F.Fab"))
-    (pad "1" thru_hole rect (at 0 0) (size 2.6 2.6) (drill 1.3) (layers "*.Cu" "*.Mask")
+    (pad "1" thru_hole rect (at 0 0 180) (size 2.6 2.6) (drill 1.3) (layers "*.Cu" "*.Mask")
       (net 15 "/X9") (pinfunction "Pin_1") (pintype "passive"))
-    (pad "2" thru_hole circle (at 5.08 0) (size 2.6 2.6) (drill 1.3) (layers "*.Cu" "*.Mask")
+    (pad "2" thru_hole circle (at 5.08 0 180) (size 2.6 2.6) (drill 1.3) (layers "*.Cu" "*.Mask")
       (net 16 "/X8") (pinfunction "Pin_2") (pintype "passive"))
     (model "${KICAD6_3DMODEL_DIR}/TerminalBlock_Phoenix.3dshapes/TerminalBlock_Phoenix_MKDS-1,5-2-5.08_1x02_P5.08mm_Horizontal.wrl"
@@
   )
   (footprint "TerminalBlock_Phoenix:TerminalBlock_Phoenix_MKDS-1,5-2-5.08_1x02_P5.08mm_Horizontal" (layer "F.Cu")
-    (at 24.7 167.14)
+    (at 107.66 138)
     (descr "Terminal Block Phoenix MKDS-1,5-2-5.08, 2 pins, pitch 5.08mm, size 10.2x9.8mm^2, drill diamater 1.3mm, pad diameter 2.6mm, see http://www.farnell.com/datasheets/100425.pdf, script-generated using https://github.com/pointhi/kicad-footprint-generator/scripts/TerminalBlock_Phoenix")
     (tags "THT Terminal Block Phoenix MKDS-1,5-2-5.08 pitch 5.08mm size 10.2x9.8mm^2 drill 1.3mm pad 2.6mm")
@@
         (effects (font (size 1 1) (thickness 0.15)))
     )
-    (fp_text value "Screw_Terminal_01x02" (at 2.54 5.66) (layer "F.Fab")
+    (fp_text value "Screw_Terminal_01x02" (at 2.54 5.66) (layer "F.Fab") hide
         (effects (font (size 1 1) (thickness 0.15)))
     )
@@
   )
   (footprint "TerminalBlock_Phoenix:TerminalBlock_Phoenix_MKDS-1,5-2-5.08_1x02_P5.08mm_Horizontal" (layer "F.Cu")
-    (at 36.92 155.28)
+    (at 102.5 62 180)
     (descr "Terminal Block Phoenix MKDS-1,5-2-5.08, 2 pins, pitch 5.08mm, size 10.2x9.8mm^2, drill diamater 1.3mm, pad diameter 2.6mm, see http://www.farnell.com/datasheets/100425.pdf, script-generated using https://github.com/pointhi/kicad-footprint-generator/scripts/TerminalBlock_Phoenix")
     (tags "THT Terminal Block Phoenix MKDS-1,5-2-5.08 pitch 5.08mm size 10.2x9.8mm^2 drill 1.3mm pad 2.6mm")
@@
         (effects (font (size 1 1) (thickness 0.15)))
     )
-    (fp_text value "W_CT_HWS" (at 2.54 5.66) (layer "F.Fab")
+    (fp_text value "W_CT_HWS" (at 2.54 5.66) (layer "F.Fab") hide
         (effects (font (size 1 1) (thickness 0.15)))
     )
@@
     (fp_circle (center 5.08 0) (end 6.58 0)
       (stroke (width 0.1) (type solid)) (fill none) (layer "F.Fab"))
-    (pad "1" thru_hole rect (at 0 0) (size 2.6 2.6) (drill 1.3) (layers "*.Cu" "*.Mask")
+    (pad "1" thru_hole rect (at 0 0 180) (size 2.6 2.6) (drill 1.3) (layers "*.Cu" "*.Mask")
       (net 11 "/X5") (pinfunction "Pin_1") (pintype "passive"))
-    (pad "2" thru_hole circle (at 5.08 0) (size 2.6 2.6) (drill 1.3) (layers "*.Cu" "*.Mask")
+    (pad "2" thru_hole circle (at 5.08 0 180) (size 2.6 2.6) (drill 1.3) (layers "*.Cu" "*.Mask")
       (net 12 "/X4") (pinfunction "Pin_2") (pintype "passive"))
     (model "${KICAD6_3DMODEL_DIR}/TerminalBlock_Phoenix.3dshapes/TerminalBlock_Phoenix_MKDS-1,5-2-5.08_1x02_P5.08mm_Horizontal.wrl"
@@
         (effects (font (size 1 1) (thickness 0.15)))
     )
-    (fp_text value "Screw_Terminal_01x02" (at 2.54 5.66) (layer "F.Fab")
+    (fp_text value "Screw_Terminal_01x02" (at 2.54 5.66) (layer "F.Fab") hide
         (effects (font (size 1 1) (thickness 0.15)))
     )
@@
         (effects (font (size 1 1) (thickness 0.15)))
     )
-    (fp_text value "Screw_Terminal_01x02" (at 2.54 5.66) (layer "F.Fab")
+    (fp_text value "Screw_Terminal_01x02" (at 2.54 5.66) (layer "F.Fab") hide
         (effects (font (size 1 1) (thickness 0.15)))
     )
@@
   )
   (footprint "TerminalBlock_Phoenix:TerminalBlock_Phoenix_MKDS-1,5-2-5.08_1x02_P5.08mm_Horizontal" (layer "F.Cu")
-    (at 36.92 143.42)
+    (at 92.34 62 180)
     (descr "Terminal Block Phoenix MKDS-1,5-2-5.08, 2 pins, pitch 5.08mm, size 10.2x9.8mm^2, drill diamater 1.3mm, pad diameter 2.6mm, see http://www.farnell.com/datasheets/100425.pdf, script-generated using https://github.com/pointhi/kicad-footprint-generator/scripts/TerminalBlock_Phoenix")
     (tags "THT Terminal Block Phoenix MKDS-1,5-2-5.08 pitch 5.08mm size 10.2x9.8mm^2 drill 1.3mm pad 2.6mm")
@@
         (effects (font (size 1 1) (thickness 0.15)))
     )
-    (fp_text value "V_ST_CWS" (at 2.54 5.66) (layer "F.Fab")
+    (fp_text value "V_ST_CWS" (at 2.54 5.66) (layer "F.Fab") hide
         (effects (font (size 1 1) (thickness 0.15)))
     )
@@
     (fp_circle (center 5.08 0) (end 6.58 0)
       (stroke (width 0.1) (type solid)) (fill none) (layer "F.Fab"))
-    (pad "1" thru_hole rect (at 0 0) (size 2.6 2.6) (drill 1.3) (layers "*.Cu" "*.Mask")
+    (pad "1" thru_hole rect (at 0 0 180) (size 2.6 2.6) (drill 1.3) (layers "*.Cu" "*.Mask")
       (net 9 "/X3") (pinfunction "Pin_1") (pintype "passive"))
-    (pad "2" thru_hole circle (at 5.08 0) (size 2.6 2.6) (drill 1.3) (layers "*.Cu" "*.Mask")
+    (pad "2" thru_hole circle (at 5.08 0 180) (size 2.6 2.6) (drill 1.3) (layers "*.Cu" "*.Mask")
       (net 10 "/X2") (pinfunction "Pin_2") (pintype "passive"))
     (model "${KICAD6_3DMODEL_DIR}/TerminalBlock_Phoenix.3dshapes/TerminalBlock_Phoenix_MKDS-1,5-2-5.08_1x02_P5.08mm_Horizontal.wrl"

Commit message: din-3u-button-panel
Parts:
- added H1: MountingHole, MountingHole:MountingHole_3.5mm, F.Cu at (120.0, 128.5)
- added H2: MountingHole, MountingHole:MountingHole_3.5mm, F.Cu at (80.0, 128.5)
- added H3: MountingHole, MountingHole:MountingHole_3.5mm, F.Cu at (80.0, 71.5)
- added H4: MountingHole, MountingHole:MountingHole_3.5mm, F.Cu at (120.0, 71.5)
- added J11: Conn_01x01_Pin, Connector_Pin:Pin_D1.0mm_L10.0mm, F.Cu at (97.2, 69.8)
- added J12: Conn_01x01_Pin, Connector_Pin:Pin_D1.0mm_L10.0mm, F.Cu at (97.0, 98.0)
- added J13: Conn_01x01_Pin, Connector_Pin:Pin_D1.0mm_L10.0mm, F.Cu at (102.5, 98.0)
- added J14: Conn_01x01_Pin, Connector_Pin:Pin_D1.0mm_L10.0mm, F.Cu at (102.2, 69.8)
- added J15: Conn_01x01_Pin, Connector_Pin:Pin_D1.0mm_L10.0mm, F.Cu at (113.0, 98.0)
- added J16: Conn_01x01_Pin, Connector_Pin:Pin_D1.0mm_L10.0mm, F.Cu at (107.5, 98.0)
- added J17: Conn_01x01_Pin, Connector_Pin:Pin_D1.0mm_L10.0mm, F.Cu at (87.4, 125.0)
- added J18: Conn_01x01_Pin, Connector_Pin:Pin_D1.0mm_L10.0mm, F.Cu at (87.4, 130.0)
- added J19: Conn_01x01_Pin, Connector_Pin:Pin_D1.0mm_L10.0mm, F.Cu at (92.5, 130.0)
- added J20: Conn_01x01_Pin, Connector_Pin:Pin_D1.0mm_L10.0mm, F.Cu at (97.5, 130.0)
- added J21: Conn_01x01_Pin, Connector_Pin:Pin_D1.0mm_L10.0mm, F.Cu at (102.6, 130.0)
- added J22: Conn_01x01_Pin, Connector_Pin:Pin_D1.0mm_L10.0mm, F.Cu at (107.7, 130.0)
- added J23: Conn_01x01_Pin, Connector_Pin:Pin_D1.0mm_L10.0mm, F.Cu at (112.8, 130.0)
- added J24: Conn_01x01_Pin, Connector_Pin:Pin_D1.0mm_L10.0mm, F.Cu at (112.8, 125.0)
- added R1: 4k7, Resistor_THT:R_Axial_DIN0207_L6.3mm_D2.5mm_P15.24mm_Horizontal, F.Cu at (92.0, 95.0)
- added R2: 4k7, Resistor_THT:R_Axial_DIN0207_L6.3mm_D2.5mm_P15.24mm_Horizontal, F.Cu at (87.0, 95.0)
- added R3: 4k7, Resistor_THT:R_Axial_DIN0207_L6.3mm_D2.5mm_P15.24mm_Horizontal, F.Cu at (97.0, 95.0)
- added R4: 4k7, Resistor_THT:R_Axial_DIN0207_L6.3mm_D2.5mm_P15.24mm_Horizontal, F.Cu at (102.5, 95.1)
- added R5: 4k7, Resistor_THT:R_Axial_DIN0207_L6.3mm_D2.5mm_P15.24mm_Horizontal, F.Cu at (113.0, 95.1)
- added R6: 4k7, Resistor_THT:R_Axial_DIN0207_L6.3mm_D2.5mm_P15.24mm_Horizontal, F.Cu at (107.5, 95.1)
- J10: value AUX_INS -> Conn_01x01_Pin; footprint TerminalBlock_Phoenix:TerminalBlock_Phoenix_MKDS-1,5-2-5.08_1x02_P5.08mm_Horizontal -> Connector_Pin:Pin_D1.0mm_L10.0mm
- J5: value Screw_Terminal_01x02 -> Conn_01x01_Pin; footprint TerminalBlock_Phoenix:TerminalBlock_Phoenix_MKDS-1,5-2-5.08_1x02_P5.08mm_Horizontal -> Connector_Pin:Pin_D1.0mm_L10.0mm
- J6: value V_ST_HWS -> Z1
- J7: value V_ST_CWS -> Z2
- J8: value W_CT_HWS -> Z3
- J9: value W_CT_CWS -> Z4
- moved J10 50.8 mm to (87.0, 98.0), turned to 0 degrees
- moved J5 47.6 mm to (92.0, 98.0)
- moved J1 5.00 mm to (82.2, 138.0)
- moved J2 5.00 mm to (92.3, 138.0)
- moved J3 5.00 mm to (102.5, 138.0)
- moved J4 5.00 mm to (112.7, 138.0)
- moved J6 5.00 mm to (87.2, 62.0)
- moved J7 5.00 mm to (97.3, 62.0)
- moved J8 5.00 mm to (107.5, 62.0)
- moved J9 5.00 mm to (117.7, 62.0)
Connections:
- J1 pad 1: /Y0 -> Net-(J1-Pin_1)
- J1 pad 2: /Y1 -> Net-(J1-Pin_2)
- J10 pad 1: /X9 -> Net-(J10-Pin_1)
- J2 pad 1: /Y2 -> Net-(J19-Pin_1)
- J2 pad 2: /Y3 -> Net-(J2-Pin_2)
- J3 pad 1: /VCC -> Net-(J21-Pin_1)
- J3 pad 2: /GND -> Net-(J22-Pin_1)
- J4 pad 1: /B -> Net-(J23-Pin_1)
- J4 pad 2: /A -> Net-(J24-Pin_1)
- J5 pad 1: /Y4 -> Net-(J5-Pin_1)
- J6 pad 1: /X1 -> Net-(J6-Pin_1)
- J6 pad 2: /X0 -> Net-(J6-Pin_2)
- J7 pad 1: /X3 -> Net-(J11-Pin_1)
- J7 pad 2: /X2 -> Net-(J7-Pin_2)
- J8 pad 1: /X5 -> Net-(J8-Pin_1)
- J8 pad 2: /X4 -> Net-(J14-Pin_1)
- J9 pad 1: /X7 -> Net-(J9-Pin_1)
- J9 pad 2: /X6 -> Net-(J9-Pin_2)
Routing:
- net Net-(J9-Pin_2): track 0.00 -> 20.0 mm
- net Net-(J8-Pin_1): track 0.00 -> 20.0 mm
- net Net-(J9-Pin_1): track 0.00 -> 19.8 mm
- net Net-(J6-Pin_2): track 0.00 -> 19.8 mm
- net Net-(J6-Pin_1): track 0.00 -> 19.8 mm
- net Net-(J7-Pin_2): track 0.00 -> 19.7 mm
- net Net-(J1-Pin_1): track 0.00 -> 15.2 mm
- net Net-(J24-Pin_1): track 0.00 -> 15.1 mm
- net Net-(J23-Pin_1): track 0.00 -> 8.00 mm
- net Net-(J22-Pin_1): track 0.00 -> 8.00 mm
- net Net-(J21-Pin_1): track 0.00 -> 8.00 mm
- net Net-(J2-Pin_2): track 0.00 -> 8.00 mm
- net Net-(J19-Pin_1): track 0.00 -> 8.00 mm
- net Net-(J1-Pin_2): track 0.00 -> 8.00 mm
- net Net-(J14-Pin_1): track 0.00 -> 7.93 mm
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Other:
- board size 64 x 84 mm -> 46 x 84 mm
