File: din-3u-button-panel/din-3u-button-panel.kicad_sch (KiCad schematic)
At the start: 11 parts, among them J1 Screw_Terminal_01x02, J10 AUX_INS, J2 Screw_Terminal_01x02, J3 Screw_Terminal_01x02, J4 Screw_Terminal_01x02, J5 Screw_Terminal_01x02, J6 V_ST_HWS, J7 V_ST_CWS, J8 W_CT_HWS, J9 W_CT_CWS

Commit message: din-3u-button-panel: update
Parts:
- J10: value AUX_INS -> Z5
- J6: value V_ST_HWS -> Z1
- J7: value V_ST_CWS -> Z2
- J8: value W_CT_HWS -> Z3
- J9: value W_CT_CWS -> Z4
Changed lines of the file:
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@@
   (symbol (lib_id "Connector:Screw_Terminal_01x02") (at 217.17 49.53 0) (unit 1)
     (in_bom yes) (on_board yes) (dnp no) (fields_autoplaced)
-    (property "Reference" "J8" (at 219.71 49.5299 0)
-      (effects (font (size 1.27 1.27)) (justify left))
-    )
-    (property "Value" "W_CT_HWS" (at 219.71 52.0699 0)
+    (property "Reference" "J8" (at 219.71 49.53 0)
+      (effects (font (size 1.27 1.27)) (justify left))
+    )
+    (property "Value" "Z3" (at 219.71 52.07 0)
       (effects (font (size 1.27 1.27)) (justify left))
     )
@@
   (symbol (lib_id "Connector:Screw_Terminal_01x02") (at 217.17 55.88 0) (unit 1)
     (in_bom yes) (on_board yes) (dnp no) (fields_autoplaced)
-    (property "Reference" "J9" (at 219.71 55.8799 0)
-      (effects (font (size 1.27 1.27)) (justify left))
-    )
-    (property "Value" "W_CT_CWS" (at 219.71 58.4199 0)
+    (property "Reference" "J9" (at 219.71 55.88 0)
+      (effects (font (size 1.27 1.27)) (justify left))
+    )
+    (property "Value" "Z4" (at 219.71 58.42 0)
       (effects (font (size 1.27 1.27)) (justify left))
     )
@@
   (symbol (lib_id "Connector:Screw_Terminal_01x02") (at 217.17 62.23 0) (unit 1)
     (in_bom yes) (on_board yes) (dnp no) (fields_autoplaced)
-    (property "Reference" "J10" (at 219.71 62.2299 0)
-      (effects (font (size 1.27 1.27)) (justify left))
-    )
-    (property "Value" "AUX_INS" (at 219.71 64.7699 0)
+    (property "Reference" "J10" (at 219.71 62.23 0)
+      (effects (font (size 1.27 1.27)) (justify left))
+    )
+    (property "Value" "Z5" (at 219.71 64.77 0)
       (effects (font (size 1.27 1.27)) (justify left))
     )
@@
   (symbol (lib_id "Connector:Screw_Terminal_01x02") (at 217.17 43.18 0) (unit 1)
     (in_bom yes) (on_board yes) (dnp no) (fields_autoplaced)
-    (property "Reference" "J7" (at 219.71 43.1799 0)
-      (effects (font (size 1.27 1.27)) (justify left))
-    )
-    (property "Value" "V_ST_CWS" (at 219.71 45.7199 0)
+    (property "Reference" "J7" (at 219.71 43.18 0)
+      (effects (font (size 1.27 1.27)) (justify left))
+    )
+    (property "Value" "Z2" (at 219.71 45.72 0)
       (effects (font (size 1.27 1.27)) (justify left))
     )
@@
   (symbol (lib_id "Connector:Screw_Terminal_01x02") (at 217.17 36.83 0) (unit 1)
     (in_bom yes) (on_board yes) (dnp no) (fields_autoplaced)
-    (property "Reference" "J6" (at 219.71 36.8299 0)
-      (effects (font (size 1.27 1.27)) (justify left))
-    )
-    (property "Value" "V_ST_HWS" (at 219.71 39.3699 0)
-      (effects (font (size 1.27 1.27)) (justify left))
-    )
+    (property "Reference" "J6" (at 219.71 36.83 0)
+      (effects (font (size 1.27 1.27)) (justify left))
+    )
+    (property "Value" "Z1" (at 219.71 39.37 0)
+      (effects (font (size 1.27 1.27)) (justify left))
+    )

Commit message: din-3u-button-panel
Parts:
- removed J10: Z5, TerminalBlock_Phoenix:TerminalBlock_Phoenix_MKDS-1,5-2-5.08_1x02_P5.08mm_Horizontal, symbol Connector:Screw_Terminal_01x02
- removed J5: Screw_Terminal_01x02, TerminalBlock_Phoenix:TerminalBlock_Phoenix_MKDS-1,5-2-5.08_1x02_P5.08mm_Horizontal, symbol Connector:Screw_Terminal_01x02
- removed S7: MOMENTARY-SWITCH-SPST-LED-PTH-12MM, mod:TACTILE_SWITCH_LED_PTH_12MM, symbol SparkFun-Switches:MOMENTARY-SWITCH-SPST-LED-PTH-12MM
- added H1, H2, H3, H4: MountingHole, MountingHole:MountingHole_3.5mm, symbol Mechanical:MountingHole
- added J10, J11, J12, J13, J14, J15, J16, J17, J18, J19, J20, J21, J22, J23, J24, J5: Conn_01x01_Pin, Connector_Pin:Pin_D1.0mm_L10.0mm, symbol Connector:Conn_01x01_Pin
- added R1, R2, R3, R4, R5, R6: 4k7, Resistor_THT:R_Axial_DIN0207_L6.3mm_D2.5mm_P15.24mm_Horizontal, symbol Device:R
Connections:
- net A: no longer names the net of J4.2 (Pin_2)
- net A: now also J24.1 (Pin_1)
- net B: no longer names the net of J4.1 (Pin_1)
- net B: now also J23.1 (Pin_1)
- net GND: no longer names the net of J3.2 (Pin_2)
- net GND: now also J22.1 (Pin_1)
- net VCC: no longer names the net of J3.1 (Pin_1)
- net VCC: now also J21.1 (Pin_1)
- net X0: no longer names the net of J6.2 (Pin_2)
- net X0: now also R2.2
- net X1: no longer names the net of J6.1 (Pin_1)
- net X1: now also R1.2
- net X2: no longer names the net of J7.2 (Pin_2)
- net X2: now also R3.2
- net X3: no longer names the net of J7.1 (Pin_1)
- net X3: now also J11.1 (Pin_1)
- net X4: no longer names the net of J8.2 (Pin_2)
- net X4: now also J14.1 (Pin_1)
- net X5: no longer names the net of J8.1 (Pin_1)
- net X5: now also R4.2
- net X6: no longer names the net of J9.2 (Pin_2)
- net X6: now also R6.2
- net X7: no longer names the net of J9.1 (Pin_1)
- net X7: now also R5.2
- net Y0: no longer names the net of J1.1 (Pin_1)
- net Y0: now also J17.1 (Pin_1)
- net Y1: no longer names the net of J1.2 (Pin_2)
- net Y1: now also J18.1 (Pin_1)
- net Y2: no longer names the net of J2.1 (Pin_1)
- net Y2: now also J19.1 (Pin_1)
- net Y3: no longer names the net of J2.2 (Pin_2)
- net Y3: now also J20.1 (Pin_1)
- new net: J10.1 (Pin_1), R2.1
- new net: J5.1 (Pin_1), R1.1
- new net: J12.1 (Pin_1), R3.1
- new net: J13.1 (Pin_1), R4.1
- new net: J16.1 (Pin_1), R6.1
- new net: J15.1 (Pin_1), R5.1
